File: 2ledblink.kicad_sch (KiCad schematic)
At the start: 10 parts, among them Q1 Q_NPN_EBC C945, Q2 Q_NPN_EBC C945

Commit message: Add files via upload
Parts:
- R1, R2: value R 220 -> R 330
Changed lines of the file:
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@@
     (in_bom yes) (on_board yes) (fields_autoplaced)
     (property "Reference" "R2" (id 0) (at 66.04 35.56 90))
-    (property "Value" "R 220" (id 1) (at 66.04 38.1 90))
+    (property "Value" "R 330" (id 1) (at 66.04 38.1 90))
     (property "Footprint" "" (id 2) (at 66.04 40.132 90)
       (effects (font (size 1.27 1.27)) hide)
@@
     (in_bom yes) (on_board yes) (fields_autoplaced)
     (property "Reference" "R1" (id 0) (at 215.9 34.29 90))
-    (property "Value" "R 220" (id 1) (at 215.9 36.83 90))
+    (property "Value" "R 330" (id 1) (at 215.9 36.83 90))
     (property "Footprint" "" (id 2) (at 215.9 42.418 90)
       (effects (font (size 1.27 1.27)) hide)
@@
     )
     (path "/bf314a8d-4e19-4773-ae14-4b5d54c2b9b9"
-      (reference "R1") (unit 1) (value "R 220") (footprint "")
+      (reference "R1") (unit 1) (value "R 330") (footprint "")
     )
     (path "/15d5b99b-0553-47c0-8482-e83f25f1267a"
-      (reference "R2") (unit 1) (value "R 220") (footprint "")
+      (reference "R2") (unit 1) (value "R 330") (footprint "")
     )
     (path "/6117f319-81aa-43cb-985b-9e705e67b705"
